File: Blinkenlights.sch (EAGLE design)
At the start: 14 parts, among them Q1 2N2222, Q2 2N2222

Commit message: 2.0.0913 Version updates
Minor modifications and tweaking
Parts:
- +, -: device adafruit:PINHD-1X1 -> IXR:PINHD-1X1CB
- Q1, Q2: device adafruit:2N2222 -> IXR:2N2222
- R1, R2, R3, R4: device IXR:RESISTOR0207/10_BIG -> IXR:RESISTOR-0207/10_BIG
Changed lines of the file:
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@@
 </classes>
 <parts>
-<part name="Q1" library="adafruit" deviceset="2N2222" device=""/>
-<part name="Q2" library="adafruit" deviceset="2N2222" device=""/>
+<part name="Q1" library="IXR" deviceset="2N2222" device=""/>
+<part name="Q2" library="IXR" deviceset="2N2222" device=""/>
 <part name="BATT" library="adafruit" deviceset="CR2032" device="SMT" value="CR2032"/>
-<part name="R1" library="IXR" deviceset="RESISTOR" device="0207/10_BIG" value="220Ω"/>
-<part name="R2" library="IXR" deviceset="RESISTOR" device="0207/10_BIG" value="100kΩ"/>
-<part name="R3" library="IXR" deviceset="RESISTOR" device="0207/10_BIG" value="100kΩ"/>
-<part name="R4" library="IXR" deviceset="RESISTOR" device="0207/10_BIG" value="220Ω"/>
+<part name="R1" library="IXR" deviceset="RESISTOR" device="-0207/10_BIG" value="220Ω"/>
+<part name="R2" library="IXR" deviceset="RESISTOR" device="-0207/10_BIG" value="100kΩ"/>
+<part name="R3" library="IXR" deviceset="RESISTOR" device="-0207/10_BIG" value="100kΩ"/>
+<part name="R4" library="IXR" deviceset="RESISTOR" device="-0207/10_BIG" value="220Ω"/>
 <part name="LED1" library="IXR" deviceset="LED" device="5MM_BIG"/>
 <part name="LED2" library="IXR" deviceset="LED" device="5MM_BIG"/>
@@
 <part name="P+1" library="SparkFun" deviceset="VCC" device=""/>
 <part name="P+2" library="SparkFun" deviceset="VCC" device=""/>
-<part name="+" library="adafruit" deviceset="PINHD-1X1" device=""/>
-<part name="-" library="adafruit" deviceset="PINHD-1X1" device=""/>
+<part name="+" library="IXR" deviceset="PINHD-1X1" device="CB"/>
+<part name="-" library="IXR" deviceset="PINHD-1X1" device="CB"/>
 <part name="GND4" library="supply1" deviceset="GND" device=""/>
 <part name="P+3" library="SparkFun" deviceset="VCC" device=""/>
